File: pcb/nilgiri_hotswap.kicad_pcb (KiCad board)
At the start: 2 copper layers, 100 x 86.8 mm, 69 parts, among them J1 USB-C, J10 BAT+, J11 BAT-, J2 USB_B_Micro, J3 ISP, SW1 SW_PUSH, SW10 SW_PUSH, SW11 SW_PUSH, SW12 SW_PUSH, SW13 SW_RESET, SW14 PWR, SW2 SW_PUSH, SW3 SW_PUSH, SW4 SW_PUSH, SW5 SW_PUSH, SW6 SW_PUSH, SW7 SW_PUSH, SW8 SW_PUSH, SW9 SW_PUSH, U1 ATmega32U4-AU, U2 ProMicro, Y1 16MHz

Commit message: moved PCBs to their dir
Parts:
- SW1, SW10, SW11, SW12, SW2, SW3, SW4, SW5, SW6, SW7, SW8, SW9: footprint kbd:CherryMX_Hotswap_v2 -> nilgiri:CherryMX_Hotswap_v2
Routing:
- net Net-(D10-Pad2): track 10.5 -> 8.67 mm
