File: pcb/nilgiri_hotswap.sch (KiCad schematic (older format))
At the start: 69 parts, among them J1 USB-C, J10 BAT+, J11 BAT-, J2 USB_B_Micro, J3 ISP, SW1 SW_PUSH, SW10 SW_PUSH, SW11 SW_PUSH, SW12 SW_PUSH, SW13 SW_RESET, SW14 PWR, SW2 SW_PUSH, SW3 SW_PUSH, SW4 SW_PUSH, SW5 SW_PUSH, SW6 SW_PUSH, SW7 SW_PUSH, SW8 SW_PUSH, SW9 SW_PUSH, U1 ATmega32U4-AU, U2 ProMicro, Y1 16MHz

Commit message: moved PCBs to their dir
Parts:
- SW1, SW10, SW11, SW12, SW2, SW3, SW4, SW5, SW6, SW7, SW8, SW9: footprint kbd:CherryMX_Hotswap_v2 -> nilgiri:CherryMX_Hotswap_v2
Changed lines of the file:
@@
 EESchema Schematic File Version 4
+LIBS:nilgiri_hotswap-cache
 EELAYER 30 0
 EELAYER END
@@
 F 0 "SW1" H 7350 1705 50  0000 C CNN
 F 1 "SW_PUSH" H 7350 1614 50  0000 C CNN
-F 2 "kbd:CherryMX_Hotswap_v2" H 7350 1450 50  0001 C CNN
+F 2 "nilgiri:CherryMX_Hotswap_v2" H 7350 1450 50  0001 C CNN
 F 3 "" H 7350 1450 50  0000 C CNN
 	1    7350 1450
@@
 F 0 "SW2" H 7350 2405 50  0000 C CNN
 F 1 "SW_PUSH" H 7350 2314 50  0000 C CNN
-F 2 "kbd:CherryMX_Hotswap_v2" H 7350 2150 50  0001 C CNN
+F 2 "nilgiri:CherryMX_Hotswap_v2" H 7350 2150 50  0001 C CNN
 F 3 "" H 7350 2150 50  0000 C CNN
 	1    7350 2150
@@
 F 0 "SW5" H 8350 2405 50  0000 C CNN
 F 1 "SW_PUSH" H 8350 2314 50  0000 C CNN
-F 2 "kbd:CherryMX_Hotswap_v2" H 8350 2150 50  0001 C CNN
+F 2 "nilgiri:CherryMX_Hotswap_v2" H 8350 2150 50  0001 C CNN
 F 3 "" H 8350 2150 50  0000 C CNN
 	1    8350 2150
@@
 F 0 "SW4" H 8350 1705 50  0000 C CNN
 F 1 "SW_PUSH" H 8350 1614 50  0000 C CNN
-F 2 "kbd:CherryMX_Hotswap_v2" H 8350 1450 50  0001 C CNN
+F 2 "nilgiri:CherryMX_Hotswap_v2" H 8350 1450 50  0001 C CNN
 F 3 "" H 8350 1450 50  0000 C CNN
 	1    8350 1450
@@
 F 0 "SW6" H 8350 3105 50  0000 C CNN
 F 1 "SW_PUSH" H 8350 3014 50  0000 C CNN
-F 2 "kbd:CherryMX_Hotswap_v2" H 8350 2850 50  0001 C CNN
+F 2 "nilgiri:CherryMX_Hotswap_v2" H 8350 2850 50  0001 C CNN
 F 3 "" H 8350 2850 50  0000 C CNN
 	1    8350 2850
@@
 F 0 "SW7" H 9300 1705 50  0000 C CNN
 F 1 "SW_PUSH" H 9300 1614 50  0000 C CNN
-F 2 "kbd:CherryMX_Hotswap_v2" H 9300 1450 50  0001 C CNN
+F 2 "nilgiri:CherryMX_Hotswap_v2" H 9300 1450 50  0001 C CNN
 F 3 "" H 9300 1450 50  0000 C CNN
 	1    9300 1450
@@
 F 0 "SW8" H 9300 2405 50  0000 C CNN
 F 1 "SW_PUSH" H 9300 2314 50  0000 C CNN
-F 2 "kbd:CherryMX_Hotswap_v2" H 9300 2150 50  0001 C CNN
+F 2 "nilgiri:CherryMX_Hotswap_v2" H 9300 2150 50  0001 C CNN
 F 3 "" H 9300 2150 50  0000 C CNN
 	1    9300 2150
@@
 F 0 "SW11" H 10300 2405 50  0000 C CNN
 F 1 "SW_PUSH" H 10300 2314 50  0000 C CNN
-F 2 "kbd:CherryMX_Hotswap_v2" H 10300 2150 50  0001 C CNN
+F 2 "nilgiri:CherryMX_Hotswap_v2" H 10300 2150 50  0001 C CNN
 F 3 "" H 10300 2150 50  0000 C CNN
 	1    10300 2150
@@
 F 0 "SW10" H 10300 1705 50  0000 C CNN
 F 1 "SW_PUSH" H 10300 1614 50  0000 C CNN
-F 2 "kbd:CherryMX_Hotswap_v2" H 10300 1450 50  0001 C CNN
+F 2 "nilgiri:CherryMX_Hotswap_v2" H 10300 1450 50  0001 C CNN
 F 3 "" H 10300 1450 50  0000 C CNN
 	1    10300 1450
@@
 F 0 "SW9" H 9300 3105 50  0000 C CNN
 F 1 "SW_PUSH" H 9300 3014 50  0000 C CNN
-F 2 "kbd:CherryMX_Hotswap_v2" H 9300 2850 50  0001 C CNN
+F 2 "nilgiri:CherryMX_Hotswap_v2" H 9300 2850 50  0001 C CNN
 F 3 "" H 9300 2850 50  0000 C CNN
 	1    9300 2850
@@
 F 0 "SW12" H 10300 3105 50  0000 C CNN
 F 1 "SW_PUSH" H 10300 3014 50  0000 C CNN
-F 2 "kbd:CherryMX_Hotswap_v2" H 10300 2850 50  0001 C CNN
+F 2 "nilgiri:CherryMX_Hotswap_v2" H 10300 2850 50  0001 C CNN
 F 3 "" H 10300 2850 50  0000 C CNN
 	1    10300 2850
@@
 F 0 "SW3" H 7350 3105 50  0000 C CNN
 F 1 "SW_PUSH" H 7350 3014 50  0000 C CNN
-F 2 "kbd:CherryMX_Hotswap_v2" H 7350 2850 50  0001 C CNN
+F 2 "nilgiri:CherryMX_Hotswap_v2" H 7350 2850 50  0001 C CNN
 F 3 "" H 7350 2850 50  0000 C CNN
 	1    7350 2850
