File: pcb/palette1202-OB.kicad_pcb (KiCad board)
At the start: 2 copper layers, 100 x 80.7 mm, 55 parts, among them J1 USB-C, J2 USB_B_Micro, J3 ISP, J4 OLED, SW1 SW_PUSH, SW10 SW_PUSH, SW11 SW_PUSH, SW12 SW_PUSH, SW2 SW_PUSH, SW20 SW_RESET, SW3 SW_PUSH, SW4 SW_PUSH, SW5 SW_PUSH, SW6 SW_PUSH, SW7 SW_PUSH, SW8 SW_PUSH, SW9 SW_PUSH, U1 ATmega32U4-AU, Y1 16MHz

Commit message: revised annotation, BOM, etc.
Parts:
- moved J3 0.10 mm to (150.4, 63.1)
- renumbered D20 to D13, D21 to D14, D30 to D20, R6 to R5
Connections:
- J1 pad S1: Net-(J1-PadS1) -> GND
- J2 pad 6: Net-(J2-Pad6) -> GND
Routing:
- net GND: track 161.4 -> 125.5 mm, vias 4 -> 8
- net VCC: track 60.7 -> 77.5 mm
- net MOSI: track 175.5 -> 166.6 mm, vias 1 -> 2
- net RB2: track 102.5 -> 98.8 mm
- net RA2: track 104.0 -> 100.4 mm
- net RESET: track 89.3 -> 91.9 mm
- net Net-(D12-Pad2): track 28.1 -> 29.9 mm
- net Net-(D6-Pad2): track 17.2 -> 15.5 mm
- net Col1: track 84.0 -> 85.2 mm
- net Net-(D1-Pad2): track 18.5 -> 19.5 mm
- net D-: track 28.7 -> 29.5 mm
- net Net-(D20-Pad1): track 45.8 -> 46.6 mm
- net RA1: track 87.3 -> 86.5 mm
- net SDA: track 40.5 -> 39.9 mm
- net MISO: track 174.7 -> 174.2 mm, vias 2 -> 1
Other:
- board text added: "OBE / v0.90(191124)"
- board text removed: "OBE / v0.50(191121)"
