File: pcb/palette1202-OB.sch (KiCad schematic (older format))
At the start: 55 parts, among them J1 USB-C, J2 USB_B_Micro, J3 ISP, J4 OLED, SW1 SW_PUSH, SW10 SW_PUSH, SW11 SW_PUSH, SW12 SW_PUSH, SW2 SW_PUSH, SW20 SW_RESET, SW3 SW_PUSH, SW4 SW_PUSH, SW5 SW_PUSH, SW6 SW_PUSH, SW7 SW_PUSH, SW8 SW_PUSH, SW9 SW_PUSH, U1 ATmega32U4-AU, Y1 16MHz

Commit message: revised annotation, BOM, etc.
Parts:
- renumbered D20 to D13, D21 to D14, D30 to D20, R6 to R5
Connections:
- net GND: now also J1.S1 (SHIELD), J2.6 (Shield)
- no-connect marks 15 -> 13
Changed lines of the file:
@@
 EESchema Schematic File Version 4
-LIBS:nilgiri 2-cache
+LIBS:palette1202-OB-cache
 EELAYER 30 0
 EELAYER END
@@
 Row1
 $Comp
-L Device:R R6
+L Device:R R5
 U 1 1 5D95E829
 P 1900 1000
-F 0 "R6" V 2107 1000 50  0000 C CNN
+F 0 "R5" V 2107 1000 50  0000 C CNN
 F 1 "10k" V 2016 1000 50  0000 C CNN
 F 2 "Resistor_SMD:R_0603_1608Metric_Pad1.05x0.95mm_HandSolder" V 1830 1000 50  0001 C CNN
@@
 	900  4350 900  4250
 $Comp
-L Device:D_Schottky D30
+L Device:D_Schottky D20
 U 1 1 5D937E12
 P 2950 1400
-F 0 "D30" V 3000 1300 50  0000 R CNN
+F 0 "D20" V 3000 1300 50  0000 R CNN
 F 1 "MBR120" V 2900 1300 50  0000 R CNN
 F 2 "Keebio:D_SOD123F" H 2950 1400 50  0001 C CNN
@@
 	9500 3950 9200 3950
 $Comp
-L Device:D D20
+L Device:D D13
 U 1 1 5D96543D
 P 7650 4150
-F 0 "D20" H 7700 4250 50  0000 R CNN
+F 0 "D13" H 7700 4250 50  0000 R CNN
 F 1 "1N4148W" H 7700 4350 50  0000 R CNN
 F 2 "nilgiri:D3_TH_SMD" H 7650 4150 50  0001 C CNN
@@
 $EndComp
 $Comp
-L Device:D D21
+L Device:D D14
 U 1 1 5D95D9B5
 P 9350 4150
-F 0 "D21" H 9400 4300 50  0000 R CNN
+F 0 "D14" H 9400 4300 50  0000 R CNN
 F 1 "1N4148W" H 9400 4400 50  0000 R CNN
 F 2 "nilgiri:D3_TH_SMD" H 9350 4150 50  0001 C CNN
@@
 Text GLabel 3450 3300 2    50   Input ~ 0
 SCL
-NoConn ~ 4350 2450
 Wire Wire Line
 	3950 4200 3450 4200
@@
 	-1   0    0    -1
 $EndComp
-NoConn ~ 4350 3800
 Wire Wire Line
 	5350 1650 5250 1650
@@
 	3950 5500 2850 5500
 Connection ~ 2850 5500
+Wire Wire Line
+	4350 2450 4650 2450
+Connection ~ 4650 2450
+Wire Wire Line
+	4350 3800 4450 3800
+Connection ~ 4450 3800
 $EndSCHEMATC
