File: pcb/palette1202-front.kicad_pcb (KiCad board)
At the start: 2 copper layers, 100 x 67.8 mm, 4 parts

Commit message: updated front panel
Parts:
- moved H8 1.41 mm to (163.6, 110.4)
- moved H6 1.00 mm to (103.1, 110.4)
- moved H7 1.00 mm to (163.6, 71.0)
