File: pcb/palette1202-PM.sch (KiCad schematic (older format))
At the start: 45 parts, among them J10 BAT+, J11 BAT-, J4 OLED, SW1 SW_PUSH, SW10 SW_PUSH, SW11 SW_PUSH, SW12 SW_PUSH, SW2 SW_PUSH, SW20 SW_RESET, SW21 PWR, SW3 SW_PUSH, SW4 SW_PUSH, SW5 SW_PUSH, SW6 SW_PUSH, SW7 SW_PUSH, SW8 SW_PUSH, SW9 SW_PUSH, U2 ProMicro

Commit message: revised annotation, BOM, etc.
Parts:
- renumbered D20 to D13, D21 to D14, D32 to D30
Changed lines of the file:
@@
 EESchema Schematic File Version 4
-LIBS:nilgiri-cache
+LIBS:palette1202-PM-cache
 EELAYER 30 0
 EELAYER END
@@
 Wire Wire Line
 	9500 3950 9200 3950
-$Comp
-L Device:D D20
-U 1 1 5D96543D
-P 7650 4150
-F 0 "D20" H 7700 4250 50  0000 R CNN
-F 1 "1N4148W" H 7700 4350 50  0000 R CNN
-F 2 "nilgiri:D3_TH_SMD" H 7650 4150 50  0001 C CNN
-F 3 "~" H 7650 4150 50  0001 C CNN
-	1    7650 4150
-	-1   0    0    1
-$EndComp
-$Comp
-L Device:D D21
-U 1 1 5D95D9B5
-P 9350 4150
-F 0 "D21" H 9400 4300 50  0000 R CNN
-F 1 "1N4148W" H 9400 4400 50  0000 R CNN
-F 2 "nilgiri:D3_TH_SMD" H 9350 4150 50  0001 C CNN
-F 3 "~" H 9350 4150 50  0001 C CNN
-	1    9350 4150
-	-1   0    0    1
-$EndComp
 Wire Wire Line
 	8400 4050 8600 4050
@@
 VCC
 $Comp
-L Device:D_Schottky D32
+L Device:D_Schottky D30
 U 1 1 5DD7EBC8
 P 4550 3350
-F 0 "D32" V 4500 3650 50  0000 R CNN
+F 0 "D30" V 4500 3650 50  0000 R CNN
 F 1 "MBR120" V 4600 3800 50  0000 R CNN
 F 2 "Keebio:D_SOD123F" H 4550 3350 50  0001 C CNN
@@
 Wire Wire Line
 	5200 3800 5200 3950
+$Comp
+L Device:D D14
+U 1 1 5D95D9B5
+P 9350 4150
+F 0 "D14" H 9400 4300 50  0000 R CNN
+F 1 "1N4148W" H 9400 4400 50  0000 R CNN
+F 2 "nilgiri:D3_TH_SMD" H 9350 4150 50  0001 C CNN
+F 3 "~" H 9350 4150 50  0001 C CNN
+	1    9350 4150
+	-1   0    0    1
+$EndComp
+$Comp
+L Device:D D13
+U 1 1 5D96543D
+P 7650 4150
+F 0 "D13" H 7700 4250 50  0000 R CNN
+F 1 "1N4148W" H 7700 4350 50  0000 R CNN
+F 2 "nilgiri:D3_TH_SMD" H 7650 4150 50  0001 C CNN
+F 3 "~" H 7650 4150 50  0001 C CNN
+	1    7650 4150
+	-1   0    0    1
+$EndComp
 $EndSCHEMATC

Commit message: updated main board
Parts:
- added C11: 100u, Capacitor_Tantalum_SMD:CP_EIA-3216-10_Kemet-I_Pad1.58x1.35mm_HandSolder, symbol Device:CP_Small
- added J20: BAT+, nilgiri:Hole 0.8mm, symbol Connector:Conn_01x01_Female
- added J21: BAT-, nilgiri:Hole 0.8mm, symbol Connector:Conn_01x01_Female
- added JP100: LEFT-A1, Jumper:SolderJumper-2_P1.3mm_Open_TrianglePad1.0x1.5mm, symbol Jumper:SolderJumper_2_Bridged
- added JP101: LEFT-B1, Jumper:SolderJumper-2_P1.3mm_Open_TrianglePad1.0x1.5mm, symbol Jumper:SolderJumper_2_Bridged
- added JP110: RIGHT-B1, Jumper:SolderJumper-2_P1.3mm_Open_TrianglePad1.0x1.5mm, symbol Jumper:SolderJumper_2_Open
- added JP111: RIGHT-A1, Jumper:SolderJumper-2_P1.3mm_Open_TrianglePad1.0x1.5mm, symbol Jumper:SolderJumper_2_Open
- added JP120: LEFT-A2, Jumper:SolderJumper-2_P1.3mm_Open_TrianglePad1.0x1.5mm, symbol Jumper:SolderJumper_2_Bridged
- added JP121: LEFT-B2, Jumper:SolderJumper-2_P1.3mm_Open_TrianglePad1.0x1.5mm, symbol Jumper:SolderJumper_2_Bridged
- added JP130: RIGHT-B2, Jumper:SolderJumper-2_P1.3mm_Open_TrianglePad1.0x1.5mm, symbol Jumper:SolderJumper_2_Open
- added JP131: RIGHT-A2, Jumper:SolderJumper-2_P1.3mm_Open_TrianglePad1.0x1.5mm, symbol Jumper:SolderJumper_2_Open
- added JP200: LEFT-SDA, Jumper:SolderJumper-2_P1.3mm_Open_TrianglePad1.0x1.5mm, symbol Jumper:SolderJumper_2_Bridged
- added JP201: LEFT-SCL, Jumper:SolderJumper-2_P1.3mm_Open_TrianglePad1.0x1.5mm, symbol Jumper:SolderJumper_2_Bridged
- added JP202: LEFT-VCC, Jumper:SolderJumper-2_P1.3mm_Open_TrianglePad1.0x1.5mm, symbol Jumper:SolderJumper_2_Bridged
- added JP203: LEFT-GND, Jumper:SolderJumper-2_P1.3mm_Open_TrianglePad1.0x1.5mm, symbol Jumper:SolderJumper_2_Bridged
- added JP210: RIGHT-SDA, Jumper:SolderJumper-2_P1.3mm_Open_TrianglePad1.0x1.5mm, symbol Jumper:SolderJumper_2_Open
- added JP211: RIGHT-SCL, Jumper:SolderJumper-2_P1.3mm_Open_TrianglePad1.0x1.5mm, symbol Jumper:SolderJumper_2_Open
- added JP212: RIGHT-VCC, Jumper:SolderJumper-2_P1.3mm_Open_TrianglePad1.0x1.5mm, symbol Jumper:SolderJumper_2_Open
- added JP213: RIGHT-GND, Jumper:SolderJumper-2_P1.3mm_Open_TrianglePad1.0x1.5mm, symbol Jumper:SolderJumper_2_Open
- added JP220: VCC-USB, Jumper:SolderJumper-2_P1.3mm_Open_TrianglePad1.0x1.5mm, symbol Jumper:SolderJumper_2_Open
- added JP221: VCC-BAT, Jumper:SolderJumper-2_P1.3mm_Open_TrianglePad1.0x1.5mm, symbol Jumper:SolderJumper_2_Open
- added SW22: PWR, Button_Switch_SMD:SW_SPDT_PCM12, symbol Switch:SW_SPDT
- D1, D10, D11, D12, D13, D14, D2, D3, D4, D5, D6, D7, D8, D9: footprint nilgiri:D3_TH_SMD -> kbd:D3_TH_SMD
- D30, D31: footprint Keebio:D_SOD123F -> kbd:D3_SMD
- SW1, SW10, SW11, SW12, SW2, SW3, SW4, SW5, SW6, SW7, SW8, SW9: footprint nilgiri:CherryMX_Choc_Hotswap-1Side -> nilgiri:CherryMX_Choc_Hotswap
- U2: footprint kbd:ProMicro_v3 -> kbd:ProMicro_v2
Connections:
- net GND: now also C11.2, J21.1 (Pin_1), JP203.1 (A), JP213.1 (A); no longer J4.4 (Pin_4)
- net RA1: now also JP100.1 (A), JP111.1 (A); no longer EC1.A
- net RA2: now also JP120.1 (A), JP131.1 (A); no longer EC2.A
- net RB1: now also JP101.1 (A), JP110.1 (A); no longer EC1.B
- net RB2: now also JP121.1 (A), JP130.1 (A); no longer EC2.B
- net SCL: now also JP201.1 (A), JP211.1 (A); no longer J4.2 (Pin_2)
- net SDA: now also JP200.1 (A), JP210.1 (A); no longer J4.1 (Pin_1)
- net VCC: now also JP220.1 (A); no longer J4.3 (Pin_3)
- net Vbat: now reaches C10.1, J10.1 (Pin_1), SW21.2 (B)
- net Vbat: now also C11.1, J20.1 (Pin_1), JP221.1 (A), SW22.2 (B)
- net at D30.1 (K), D31.1 (K), SW21.1 (A): now also SW22.1 (A)
- new net: EC1.A, JP100.2 (B), JP110.2 (B)
- new net: EC1.B, JP101.2 (B), JP111.2 (B)
- new net: EC2.A, JP120.2 (B), JP130.2 (B)
- new net: EC2.B, JP121.2 (B), JP131.2 (B)
- new net: J4.1 (Pin_1), JP200.2 (B), JP213.2 (B)
- new net: J4.2 (Pin_2), JP201.2 (B), JP212.2 (B)
- new net: J4.3 (Pin_3), JP202.2 (B), JP211.2 (B)
- new net: J4.4 (Pin_4), JP203.2 (B), JP210.2 (B)
- new net: JP202.1 (A), JP212.1 (A), JP220.2 (B), JP221.2 (B)
- no-connect marks 6 -> 7
Other:
- moved on the sheet: BT1, BT2, C10, D14, D30, D31, EC2, J10, J11, J4, SW20, SW21

Commit message: added connecter for split layout(testing)
Parts:
- added J1_LEFT1, J2_RIGHT1: AudioJack4, Connector_Audio:Jack_3.5mm_PJ320E_Horizontal, symbol Connector:AudioJack4
- SW1, SW10, SW11, SW12, SW2, SW3, SW4, SW5, SW6, SW7, SW8, SW9: symbol kbd:SW_PUSH -> palette1202-PM-rescue:SW_PUSH-kbd
- U2: symbol kbd:ProMicro -> palette1202-PM-rescue:ProMicro-kbd
Connections:
- net GND: now also J1_LEFT1.S, J2_RIGHT1.S
- net VCC: now also J1_LEFT1.T, J2_RIGHT1.T
- net DATA: now reaches U2.1 (TX0/D3)
- net DATA: now also J1_LEFT1.R1, J1_LEFT1.R2, J2_RIGHT1.R1, J2_RIGHT1.R2
- net LEFT: now reaches U2.2 (RX1/D2)
- net LEFT: now also JP202.1 (A), JP212.1 (A), JP220.2 (B), JP221.2 (B)
- no-connect marks 7 -> 5
